File: kicad/ltdc.kicad_sch (KiCad schematic)
At the start: 0 parts

Commit message: many updates
Other:
- note added: "find connector?"
- note added: "or find display"
Changed lines of the file:
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@@
+		)
+	)
+	(text "or find display"
+		(exclude_from_sim no)
+		(at 122.174 66.294 0)
+		(effects
+			(font
+				(size 1.27 1.27)
+			)
+		)
+	)
+	(text "find connector?"
+		(exclude_from_sim no)
+		(at 122.936 53.848 0)
+		(effects
+			(font
+				(size 1.27 1.27)
+			)
 		)
 	)
