File: kicad/ulpi.kicad_sch (KiCad schematic)
At the start: 17 parts, among them U10 TPD3S014, U11 USB3300-EZK, X4 24MHz

Commit message: many updates
Parts:
- removed C56, C57: C_Small, symbol Device:C_Small
- removed X4: 24MHz, symbol Crystal_AKL:Crystal_Generic_GND24
- C46: renamed from C48; footprint (none) -> Capacitor_SMD:C_0603_1608Metric
- C47: renamed from C49; footprint (none) -> Capacitor_SMD:C_0603_1608Metric
- C48: renamed from C50; footprint (none) -> Capacitor_SMD:C_0603_1608Metric
- C49: renamed from C51; footprint (none) -> Capacitor_SMD:C_0603_1608Metric
- C50: renamed from C52; footprint (none) -> Capacitor_SMD:C_0603_1608Metric
- C51: renamed from C53; footprint (none) -> Capacitor_SMD:C_0603_1608Metric
- C52: renamed from C54; footprint (none) -> Capacitor_SMD:C_0603_1608Metric
- C53: renamed from C55; footprint (none) -> Capacitor_SMD:C_0603_1608Metric
- R17, R18, R19: footprint (none) -> Resistor_SMD:R_0603_1608Metric
- renumbered TP1 to TP2
Connections:
- net ULPI_X+ renamed CLKIN
- net ULPI_X-: no longer names the net of U11.27 (XO)
- no-connect marks 2 -> 3
Other:
- note added: "check if clock is correct"
- note removed: "Crystal"
