File: kicad/audio.kicad_sch (KiCad schematic)
At the start: 14 parts, among them U9 CS4344

Commit message: many updates
Parts:
- added J5: AudioJack3, Connector_Audio:Jack_3.5mm_CUI_SJ-3523-SMT_Horizontal, symbol Connector_Audio:AudioJack3
- C38: renamed from C40; footprint (none) -> Capacitor_SMD:C_0603_1608Metric
- C39: renamed from C41; footprint (none) -> Capacitor_SMD:C_0603_1608Metric
- C40: renamed from C42; footprint (none) -> Capacitor_SMD:C_0603_1608Metric
- C41: renamed from C43; footprint (none) -> Capacitor_SMD:C_0603_1608Metric
- C42: renamed from C44; footprint (none) -> Capacitor_SMD:C_0603_1608Metric
- C43: renamed from C45; footprint (none) -> Capacitor_SMD:C_0603_1608Metric
- C44: renamed from C46; footprint (none) -> Capacitor_SMD:C_0603_1608Metric
- C45: renamed from C47; footprint (none) -> Capacitor_SMD:C_0603_1608Metric
- R13, R14, R15, R16: footprint (none) -> Resistor_SMD:R_0603_1608Metric
Other:
- note added: "3.5mm trs stereo"

Commit message: school wifi broken
Parts:
- added C73: 0.1uF, Capacitor_SMD:C_0603_1608Metric, symbol Device:C_Small
- added MIC1: MMICT390200012, easyeda2kicad:MIC-SMD_5P-L3.5-W2.7-TL_MMICT390200012, symbol easyeda2kicad:MMICT390200012
Connections:
- net +3.3V: now also C73.1, MIC1.5 (VDD)
- net AOUTL: now also J5.T
- net AOUTR: now also J5.R
- net GND: now also J5.S, C73.2, MIC1.3 (GND)
- new net DFSDM1.CKIN1: MIC1.4 (CLK)
- new net DFSDM1.DATIN1: MIC1.1 (DATA)
- no-connect marks 1 -> 2
Other:
- note added: "Left/Right channel select pin"
- note added: "pdm mic soon"
