File: kicad/clock.kicad_sch (KiCad schematic)
At the start: 22 parts, among them X3 TCXO, Y1 Si5351C-B-GM

Commit message: school wifi broken
Parts:
- added TP3, TP4, TP5, TP6, TP7: TestPoint, TestPoint:TestPoint_Pad_D1.5mm, symbol Connector:TestPoint
Connections:
- net at R30.2: now also TP3.1
- net at R31.2: now also TP5.1
- net at R32.2: now also TP7.1
- net at R28.2: now also TP6.1
- net at R27.2: now also TP4.1
