File: kicad/ethernet.kicad_sch (KiCad schematic)
At the start: 13 parts, among them J3 RJ45_Halo_HFJ11-x2450E-LxxRL, U8 LAN8742A, X3 25MHz

Commit message: many updates
Parts:
- removed C34, C37: 30pF, symbol Device:C_Small
- removed X3: 25MHz, symbol Crystal_AKL:Crystal_Generic_GND24
- C34: renamed from C35; footprint (none) -> Capacitor_SMD:C_0603_1608Metric
- C35: renamed from C36; footprint (none) -> Capacitor_SMD:C_0603_1608Metric
- C36: renamed from C38; footprint (none) -> Capacitor_SMD:C_0603_1608Metric
- R7, R8, R9: footprint (none) -> Resistor_SMD:R_0603_1608Metric
Connections:
- net CLKIN: now reaches U8.5 (XTAL1/CLKIN)
- no-connect marks 1 -> 2
Other:
- note added: "check if this is correct"
- moved on the sheet: R7, R8

Commit message: school wifi broken
Parts:
- added C92, C93, C94, C95, C96: 0.1uF, Capacitor_SMD:C_0603_1608Metric, symbol Device:C_Small
Connections:
- net +3.3V: now also C92.1, C93.1, C94.1, C95.1, C96.1
- net GND: now also C92.2, C93.2, C94.2, C95.2, C96.2
- net TD+: now reaches J3.1 (TD+), U8.21 (TXP)
- net TD-: now reaches J3.2 (TD-), U8.20 (TXN)
- net RD+: now reaches J3.3 (RD+), U8.23 (RXP)
- net RD-: now reaches J3.6 (RD-), U8.22 (RXN)
Other:
- note added: "check this pin out"
