File: kicad/power.kicad_sch (KiCad schematic)
At the start: 29 parts, among them U4 TLV75733PDBV, U5 TLV75725PDBV, U6 TLV75718PDBV, U7 TLV75712PDBV

Commit message: many updates
Parts:
- C12, C13, C14, C15, C16, C17, C18, C19, C20, C21, C22, C23, C24, C25, C26, C27, C28, C29, C30, C31, C32, C33: footprint (none) -> Capacitor_SMD:C_0603_1608Metric
- FB1, FB2, FB3: footprint (none) -> Ferrite_SMD_AKL:Ferrite_0603_1608Metric
Connections:
- net +5V: no longer U5.3 (EN), U6.3 (EN), U7.3 (EN)
- new net 1.2V_EN: U7.3 (EN)
- new net 1.8V_EN: U6.3 (EN)
- new net 2.5V_EN: U5.3 (EN)
Other:
- note removed: "add fpga power sequencing"
- note removed: "or mcu control en"
Changed lines of the file:
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@@
 		)
 	)
-	(text "add fpga power sequencing"
-		(exclude_from_sim no)
-		(at 152.3315 91.2822 0)
-		(effects
-			(font
-				(size 1.27 1.27)
-			)
-		)
-	)
 	(text "FPGA filter"
 		(exclude_from_sim no)
@@
 		)
 	)
-	(text "or mcu control en"
-		(exclude_from_sim no)
-		(at 151.638 95.504 0)
-		(effects
-			(font
-				(size 1.27 1.27)
-			)
-		)
-	)
 	(text "FPGA filter"
 		(exclude_from_sim no)
@@
 	)
 	(junction
-		(at 64.77 114.3)
-		(diameter 0)
-		(color 0 0 0 0)
-	)
-	(junction
-		(at 64.77 152.4)
-		(diameter 0)
-		(color 0 0 0 0)
-	)
-	(junction
 		(at 93.98 38.1)
 		(diameter 0)
@@
 	)
 	(junction
-		(at 64.77 76.2)
-		(diameter 0)
-		(color 0 0 0 0)
-	)
-	(junction
 		(at 82.55 87.63)
 		(diameter 0)
@@
 	(wire
 		(pts
-			(xy 66.04 78.74) (xy 64.77 78.74)
-		)
-		(stroke
-			(width 0)
-			(type default)
-		)
-	)
-	(wire
-		(pts
 			(xy 73.66 48.26) (xy 73.66 49.53)
 		)
@@
 	(wire
 		(pts
-			(xy 66.04 76.2) (xy 64.77 76.2)
+			(xy 58.42 76.2) (xy 66.04 76.2)
 		)
 		(stroke
@@
 	(wire
 		(pts
-			(xy 66.04 114.3) (xy 64.77 114.3)
+			(xy 58.42 114.3) (xy 66.04 114.3)
 		)
 		(stroke
@@
 	(wire
 		(pts
-			(xy 64.77 152.4) (xy 58.42 152.4)
+			(xy 66.04 78.74) (xy 64.77 78.74)
 		)
 		(stroke
@@
 	(wire
 		(pts
-			(xy 64.77 114.3) (xy 64.77 116.84)
+			(xy 58.42 152.4) (xy 66.04 152.4)
 		)
 		(stroke
@@
 	(wire
 		(pts
-			(xy 66.04 152.4) (xy 64.77 152.4)
+			(xy 64.77 111.76) (xy 64.77 116.84)
 		)
 		(stroke
@@
 	(wire
 		(pts
-			(xy 64.77 76.2) (xy 58.42 76.2)
-		)
-		(stroke
-			(width 0)
-			(type default)
-		)
-	)
-	(wire
-		(pts
 			(xy 207.01 34.29) (xy 207.01 33.02)
 		)
@@
 	(wire
 		(pts
-			(xy 64.77 114.3) (xy 58.42 114.3)
-		)
-		(stroke
-			(width 0)
-			(type default)
-		)
-	)
-	(wire
-		(pts
 			(xy 82.55 49.53) (xy 73.66 49.53)
 		)
@@
 	(wire
 		(pts
-			(xy 64.77 152.4) (xy 64.77 154.94)
+			(xy 64.77 149.86) (xy 64.77 154.94)
 		)
 		(stroke
@@
 	(wire
 		(pts
-			(xy 207.01 40.64) (xy 207.01 41.91)
+			(xy 64.77 78.74) (xy 64.77 73.66)
 		)
 		(stroke
@@
 	(wire
 		(pts
-			(xy 82.55 77.47) (xy 82.55 76.2)
+			(xy 207.01 40.64) (xy 207.01 41.91)
 		)
 		(stroke
@@
 	(wire
 		(pts
-			(xy 93.98 82.55) (xy 93.98 87.63)
+			(xy 82.55 77.47) (xy 82.55 76.2)
 		)
 		(stroke
@@
 	(wire
 		(pts
-			(xy 93.98 74.93) (xy 93.98 76.2)
+			(xy 93.98 82.55) (xy 93.98 87.63)
 		)
 		(stroke
@@
 	(wire
 		(pts
-			(xy 58.42 152.4) (xy 46.99 152.4)
+			(xy 93.98 74.93) (xy 93.98 76.2)
 		)
 		(stroke
@@
 	(wire
 		(pts
-			(xy 81.28 76.2) (xy 82.55 76.2)
+			(xy 58.42 152.4) (xy 46.99 152.4)
 		)
 		(stroke
@@
 	(wire
 		(pts
-			(xy 35.56 114.3) (xy 35.56 152.4)
+			(xy 81.28 76.2) (xy 82.55 76.2)
 		)
 		(stroke
@@
 	(wire
 		(pts
-			(xy 35.56 76.2) (xy 35.56 114.3)
+			(xy 35.56 114.3) (xy 35.56 152.4)
 		)
 		(stroke
@@
 	(wire
 		(pts
-			(xy 64.77 76.2) (xy 64.77 78.74)
+			(xy 35.56 76.2) (xy 35.56 114.3)
 		)
 		(stroke
@@
 		)
 	)
+	(hierarchical_label "1.2V_EN"
+		(shape input)
+		(at 64.77 149.86 90)
+		(effects
+			(font
+				(size 1.27 1.27)
+			)
+			(justify left)
+		)
+	)
+	(hierarchical_label "1.8V_EN"
+		(shape input)
+		(at 64.77 111.76 90)
+		(effects
+			(font
+				(size 1.27 1.27)
+			)
+			(justify left)
+		)
+	)
+	(hierarchical_label "2.5V_EN"
+		(shape input)
+		(at 64.77 73.66 90)
+		(effects
+			(font
+				(size 1.27 1.27)
+			)
+			(justify left)
+		)
+	)
 	(symbol
 		(lib_id "Device:C_Small")
@@
 			)
 		)
-		(property "Footprint" ""
+		(property "Footprint" "Capacitor_SMD:C_0603_1608Metric"
 			(at 58.42 41.91 0)
 			(hide yes)
@@
 			)
 		)
-		(property "Footprint" ""
+		(property "Footprint" "Capacitor_SMD:C_0603_1608Metric"
 			(at 93.98 156.21 0)
 			(hide yes)
@@
 			)
 		)
-		(property "Footprint" ""
+		(property "Footprint" "Capacitor_SMD:C_0603_1608Metric"
 			(at 182.88 38.1 0)
 			(hide yes)
@@
 			)
 		)
-		(property "Footprint" ""
+		(property "Footprint" "Capacitor_SMD:C_0603_1608Metric"
 			(at 82.55 41.91 0)
 			(hide yes)
@@
 			)
 		)
-		(property "Footprint" ""
+		(property "Footprint" "Ferrite_SMD_AKL:Ferrite_0603_1608Metric"
 			(at 219.71 36.068 90)
 			(hide yes)
@@
 			)
 		)
-		(property "Footprint" ""
+		(property "Footprint" "Capacitor_SMD:C_0603_1608Metric"
 			(at 46.99 156.21 0)
 			(hide yes)
@@
 			)
 		)
-		(property "Footprint" ""
+		(property "Footprint" "Capacitor_SMD:C_0603_1608Metric"
 			(at 93.98 118.11 0)
 			(hide yes)
@@
 			)
 		)
-		(property "Footprint" ""
+		(property "Footprint" "Capacitor_SMD:C_0603_1608Metric"
 			(at 257.81 38.1 0)
 			(hide yes)
@@
 			)
 		)
-		(property "Footprint" ""
+		(property "Footprint" "Capacitor_SMD:C_0603_1608Metric"
 			(at 58.42 118.11 0)
 			(hide yes)
@@
 			)
 		)
-		(property "Footprint" ""
+		(property "Footprint" "Capacitor_SMD:C_0603_1608Metric"
 			(at 82.55 80.01 0)
 			(hide yes)
@@
 			)
 		)
-		(property "Footprint" ""
+		(property "Footprint" "Capacitor_SMD:C_0603_1608Metric"
 			(at 46.99 118.11 0)
 			(hide yes)
@@
 			)
 		)
-		(property "Footprint" ""
+		(property "Footprint" "Capacitor_SMD:C_0603_1608Metric"
 			(at 46.99 80.01 0)
 			(hide yes)
@@
 			)
 		)
-		(property "Footprint" ""
+		(property "Footprint" "Capacitor_SMD:C_0603_1608Metric"
 			(at 207.01 38.1 0)
 			(hide yes)
@@
 			)
 		)
-		(property "Footprint" ""
+		(property "Footprint" "Ferrite_SMD_AKL:Ferrite_0603_1608Metric"
 			(at 270.51 36.068 90)
 			(hide yes)
@@
 			)
 		)
-		(property "Footprint" ""
+		(property "Footprint" "Capacitor_SMD:C_0603_1608Metric"
 			(at 93.98 80.01 0)
 			(hide yes)
@@
 			)
 		)
-		(property "Footprint" ""
+		(property "Footprint" "Ferrite_SMD_AKL:Ferrite_0603_1608Metric"
 			(at 168.91 36.068 90)
 			(hide yes)
@@
 			)
 		)
-		(property "Footprint" ""
+		(property "Footprint" "Capacitor_SMD:C_0603_1608Metric"
 			(at 82.55 156.21 0)
 			(hide yes)
@@
 			)
 		)
-		(property "Footprint" ""
+		(property "Footprint" "Capacitor_SMD:C_0603_1608Metric"
 			(at 284.48 38.1 0)
 			(hide yes)
@@
 			)
 		)
-		(property "Footprint" ""
+		(property "Footprint" "Capacitor_SMD:C_0603_1608Metric"
 			(at 93.98 41.91 0)
 			(hide yes)
@@
 			)
 		)
-		(property "Footprint" ""
+		(property "Footprint" "Capacitor_SMD:C_0603_1608Metric"
 			(at 58.42 156.21 0)
 			(hide yes)
@@
 			)
 		)
-		(property "Footprint" ""
+		(property "Footprint" "Capacitor_SMD:C_0603_1608Metric"
 			(at 46.99 41.91 0)
 			(hide yes)
@@
 			)
 		)
-		(property "Footprint" ""
+		(property "Footprint" "Capacitor_SMD:C_0603_1608Metric"
 			(at 156.21 38.1 0)
 			(hide yes)
@@
 			)
 		)
-		(property "Footprint" ""
+		(property "Footprint" "Capacitor_SMD:C_0603_1608Metric"
 			(at 58.42 80.01 0)
 			(hide yes)
@@
 			)
 		)
-		(property "Footprint" ""
+		(property "Footprint" "Capacitor_SMD:C_0603_1608Metric"
 			(at 233.68 38.1 0)
 			(hide yes)
@@
 			)
 		)
-		(property "Footprint" ""
+		(property "Footprint" "Capacitor_SMD:C_0603_1608Metric"
 			(at 82.55 118.11 0)
 			(hide yes)

Commit message: school wifi broken
Changed lines of the file:
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@@
 	(wire
 		(pts
-			(xy 46.99 152.4) (xy 35.56 152.4)
+			(xy 35.56 152.4) (xy 46.99 152.4)
 		)
 		(stroke
