File: kicad/STM32H743.kicad_sch (KiCad schematic)
At the start: 0 parts

Commit message: many updates
Other:
- added sheet Clock (clock.kicad_sch)
- sheet Connector ports: added ADC1{INP1 INP2 INP12 INN12}, ADC2{INN2}, ADC3{INP5 INN5 INP4}, COMP2{INP INN}, DAC1_OUT1, DCMI{D[7..0] HSYNC VSYNC PIXCLK}, FDCAN1{RX TX}, I2S2{MCK WS CK SDI SDO}, OPAMP2{VOUT VIN-}, QUADSPI{D[4..0] CLK ~{CS}}, RTC{ALARM TAMP2 CALIB}, SAI1A{MCLK FS SCK SD}, SPI4{~{CS} SCK MISO MOSI}, TIM8_CH1, USART1{TX RX CK}, USART2{TX RX}, USART3{TX RX CK}, USART6{CK TX RX}; removed I2C1{SCL SDA}
- sheet Ethernet ports: added CLKIN, RMII{CRS_DV MDIO MDC}, RMII{TXD0 TXD1 TXEN RXD0 RXD1}; removed RMII{TXD0 TXD1 TXEN RXD0 RXD1 CRS_DV MDIO MDC}
- sheet FPGA ports: added CLKIN; removed none
- sheet MCU ports: added RMII{CRS_DV MDIO MDC}, RMII{TXD0 TXD1 TXEN RXD0 RXD1}; removed HDMI_CEC, RMII{TXD0 TXD1 TXEN RXD0 RXD1 CRS_DV MDIO MDC}
- sheet Power ports: added 1.2V_EN, 1.8V_EN, 2.5V_EN; removed none
- sheet ULPI ports: added CLKIN; removed none
- sheet uSD ports: added ~{SD_DET}; removed SD_DET
- note added: "for special mic"
- note removed: "Si5351C?"
- note removed: "really need to solve clock issues"
- note removed: "too many crystals"

Commit message: school wifi broken
Parts:
- added H1, H2: MountingHole, MountingHole:MountingHole_3.2mm_M3, symbol Mechanical:MountingHole
Other:
- added sheet GPIO (gpio.kicad_sch)
- added sheet LEDs (leds.kicad_sch)
- sheet Audio ports: added DFSDM1{CKIN1 DATIN1}; removed none
- sheet FPGA ports: added FPGA{BANK0}; removed none
- sheet MCU ports: added 1.2V_EN, 1.8V_EN, 2.5V_EN, FPGA_ACT, FPGA_FAULT, FPGA{~{CRESET} CDONE}, MCU_ACT, MCU_FAULT, PB6, PF2, PG15, PG2, PG3, PG4, PG5, PH5, PH6, PH7, PI12, PI13, PJ11, PJ9, PK2, ULPI_RESET, ~{RMII_RST}, ~{SD_DET}; removed none
- note removed: "for special mic"

Commit message: blenders
Other:
- sheet FPGA ports: added BANK0_IOT{36b 37a 38b 39a 41a 42b 43a 44b 45a 46b 48b 49a 50b 51a}, BANK1_IOB{13b 16a 18a 20a 22a 23b 24a 29b 31b}, BANK2_IOB{0a 2a 3b 4a 5b 6a 8a 9b}; removed FPGA{BANK0}
- sheet GPIO ports: added BANK0_IOT{36b 37a 38b 39a 41a 42b 43a 44b 45a 46b 48b 49a 50b 51a}, BANK1_IOB{13b 16a 18a 20a 22a 23b 24a 29b 31b}, BANK2_IOB{0a 2a 3b 4a 5b 6a 8a 9b}, FPGA{~{CRESET} CDONE}, PB{6}, PF{2}, PG{[2..5] 15}, PH{[5..7]}, PI{12 13}, PJ{9 11}, PK{2}; removed FPGA{BANK0}, PB6, PF2, PG15, PG2, PG3, PG4, PG5, PH5, PH6, PH7, PI12, PI13, PJ11, PJ9, PK2
- sheet MCU ports: added PB{6}, PF{2}, PG{[2..5] 15}, PH{[5..7]}, PI{12 13}, PJ{9 11}, PK{2}; removed PB6, PF2, PG15, PG2, PG3, PG4, PG5, PH5, PH6, PH7, PI12, PI13, PJ11, PJ9, PK2
