File: kicad/connector.kicad_sch (KiCad schematic)
At the start: 1 part, among them J5 Conn_02x05_Counter_Clockwise

Commit message: many updates
Parts:
- renumbered J5 to J6

Commit message: blenders
Parts:
- added J9: Conn_02x05_Odd_Even, Connector_PinHeader_2.54mm:PinHeader_2x05_P2.54mm_Vertical, symbol Connector_Generic:Conn_02x05_Odd_Even
Connections:
- net +3.3V: now also J9.7 (Pin_7), J9.8 (Pin_8)
- net +5V: now also J9.10 (Pin_10), J9.9 (Pin_9)
- net GND: now also J9.3 (Pin_3), J9.4 (Pin_4)
- net NRST: now also J9.1 (Pin_1)
- new net SWCLK: J9.6 (Pin_6)
- new net SWDIO: J9.2 (Pin_2)
- no-connect marks 0 -> 1
Other:
- note added: "Analog"
- note added: "NO CONNECTORS FOR V1!!"
- note added: "SWD"
- note added: "audio"
- note added: "boot"
- note added: "camera"
- note added: "can bus"
- note added: "i2c bus"
- note added: "power"
- note added: "serial"
- note added: "spi"
- note added: "timekeeping"
- note added: "timer"
- note added: "xternal mem"
