File: kicad/fpga.kicad_sch (KiCad schematic)
At the start: 7 parts, among them U12 ICE40UP5K-SG48ITR, Y1 SG-210STF 12MHz

Commit message: many updates
Parts:
- removed C61: 0.1uF, symbol Device:C_Small
- removed Y1: SG-210STF 12MHz, Oscillator:Oscillator_SMD_SeikoEpson_SG210-4Pin_2.5x2.0mm, symbol Oscillator:SG-210STF
- C54: renamed from C58; footprint (none) -> Capacitor_SMD:C_0603_1608Metric
- C55: renamed from C59; footprint (none) -> Capacitor_SMD:C_0603_1608Metric
- C56: renamed from C60; footprint (none) -> Capacitor_SMD:C_0603_1608Metric
- FB4: footprint (none) -> Ferrite_SMD_AKL:Ferrite_0603_1608Metric
Connections:
- net FPGA_CLK renamed CLKIN
- no-connect marks 1 -> 0
Other:
- note removed: "Clock"

Commit message: school wifi broken
Parts:
- added C100, C101, C97, C98, C99: 0.1uF, Capacitor_SMD:C_0603_1608Metric, symbol Device:C_Small
- added D11: LED_ABGR, LED_SMD:LED_Cree-PLCC4_2x2mm_CW, symbol Device:LED_ABGR
- added RN3: 0, Resistor_SMD_AKL:R_Array_Concave_4x0603, symbol Resistor_US_AKL:R_4x0603_Concave
Connections:
- net +3.3VFPGA: now also C100.1, C101.1, C97.1, C98.1, C99.1, D11.1 (A)
- net GND: now also C100.2, C101.2, C97.2, C98.2, C99.2
- net SPI1.MISO: now also RN3.1 (R1.1); no longer U12.14 (IOB_32a_SPI_SO)
- net SPI1.MOSI: now also RN3.4 (R4.1); no longer U12.17 (IOB_33b_SPI_SI)
- net SPI1.NSS: now also RN3.3 (R3.1); no longer U12.16 (IOB_35b_SPI_SS)
- net SPI1.SCK: now also RN3.2 (R2.1); no longer U12.15 (IOB_34a_SPI_SCK)
- net BANK0_IOT_37a: now reaches U12.23 (IOT_37a)
- net BANK0_IOT_36b: now reaches U12.25 (IOT_36b)
- net BANK0_IOT_39a: now reaches U12.26 (IOT_39a)
- net BANK0_IOT_38b: now reaches U12.27 (IOT_38b)
- net BANK0_IOT_41a: now reaches U12.28 (IOT_41a)
- net BANK0_IOT_42b: now reaches U12.31 (IOT_42b)
- net BANK0_IOT_43a: now reaches U12.32 (IOT_43a)
- net BANK0_IOT_44b: now reaches U12.34 (IOT_44b)
- net BANK0_IOT_46b_G0: now reaches U12.35 (IOT_46b_G0)
- net BANK0_IOT_48b: now reaches U12.36 (IOT_48b)
- net BANK0_IOT_45a_G1: now reaches U12.37 (IOT_45a_G1)
- net BANK0_IOT_50b: now reaches U12.38 (IOT_50b)
- net at U12.39 (RGB0): now also D11.4 (RK)
- net at U12.40 (RGB1): now also D11.3 (GK)
- net at U12.41 (RGB2): now also D11.2 (BK)
- net BANK0_IOT_51a: now reaches U12.42 (IOT_51a)
- net BANK0_IOT_49a: now reaches U12.43 (IOT_49a)
- new net: RN3.8 (R1.2), U12.14 (IOB_32a_SPI_SO)
- new net: RN3.7 (R2.2), U12.15 (IOB_34a_SPI_SCK)
- new net: RN3.6 (R3.2), U12.16 (IOB_35b_SPI_SS)
- new net: RN3.5 (R4.2), U12.17 (IOB_33b_SPI_SI)
Other:
- note added: "decoupling"
- moved on the sheet: U12A

Commit message: blenders
Connections:
- net BANK1_IOB.18a: now reaches U12.10 (IOB_18a)
- net BANK1_IOB.20a: now reaches U12.11 (IOB_20a)
- net BANK1_IOB.22a: now reaches U12.12 (IOB_22a)
- net BANK1_IOB.24a: now reaches U12.13 (IOB_24a)
- net BANK1_IOB.31b: now reaches U12.18 (IOB_31b)
- net BANK1_IOB.29b: now reaches U12.19 (IOB_29b)
- net BANK1_IOB.23b: now reaches U12.21 (IOB_23b)
- net BANK1_IOB.13b: now reaches U12.6 (IOB_13b)
- net BANK1_IOB.16a: now reaches U12.9 (IOB_16a)
- net BANK2_IOB.6a: now reaches U12.2 (IOB_6a)
- net BANK2_IOB.9b: now reaches U12.3 (IOB_9b)
- net BANK2_IOB.8a: now reaches U12.4 (IOB_8a)
- net BANK2_IOB.3b: now reaches U12.44 (IOB_3b_G6)
- net BANK2_IOB.5b: now reaches U12.45 (IOB_5b)
- net BANK2_IOB.0a: now reaches U12.46 (IOB_0a)
- net BANK2_IOB.2a: now reaches U12.47 (IOB_2a)
- net BANK2_IOB.4a: now reaches U12.48 (IOB_4a)
- net BANK0_IOT_36b renamed BANK0_IOT.36b
- net BANK0_IOT_37a renamed BANK0_IOT.37a
- net BANK0_IOT_38b renamed BANK0_IOT.38b
- net BANK0_IOT_39a renamed BANK0_IOT.39a
- net BANK0_IOT_41a renamed BANK0_IOT.41a
- net BANK0_IOT_42b renamed BANK0_IOT.42b
- net BANK0_IOT_43a renamed BANK0_IOT.43a
- net BANK0_IOT_44b renamed BANK0_IOT.44b
- net BANK0_IOT_45a_G1 renamed BANK0_IOT.45a
- net BANK0_IOT_46b_G0 renamed BANK0_IOT.46b
- net BANK0_IOT_48b renamed BANK0_IOT.48b
- net BANK0_IOT_49a renamed BANK0_IOT.49a
- net BANK0_IOT_50b renamed BANK0_IOT.50b
- net BANK0_IOT_51a renamed BANK0_IOT.51a
Other:
- moved on the sheet: D11, RN3, U12A, U12B, U12C
