File: kicad/gpio.kicad_sch (KiCad schematic)
At the start: 2 parts, among them J7 Conn_02x22_Odd_Even, J8 Conn_02x10_Odd_Even

Commit message: blenders
Connections:
- net +3.3V: now also J7.20 (Pin_20), J7.22 (Pin_22), J7.24 (Pin_24), J7.26 (Pin_26), J7.28 (Pin_28)
- net GND: now also J7.34 (Pin_34), J7.36 (Pin_36), J7.38 (Pin_38), J7.40 (Pin_40), J7.42 (Pin_42), J7.44 (Pin_44)
- net PF2: no longer J8.5 (Pin_5)
- net BANK0_IOT.36b: now reaches J7.1 (Pin_1)
- net BANK1_IOB.22a: now reaches J7.10 (Pin_10)
- net BANK0_IOT.42b: now reaches J7.11 (Pin_11)
- net BANK1_IOB.23b: now reaches J7.12 (Pin_12)
- net BANK0_IOT.43a: now reaches J7.13 (Pin_13)
- net BANK1_IOB.24a: now reaches J7.14 (Pin_14)
- net BANK0_IOT.44b: now reaches J7.15 (Pin_15)
- net BANK1_IOB.29b: now reaches J7.16 (Pin_16)
- net BANK0_IOT.45a: now reaches J7.17 (Pin_17)
- net BANK1_IOB.31b: now reaches J7.18 (Pin_18)
- net BANK0_IOT.46b: now reaches J7.19 (Pin_19)
- net BANK1_IOB.13b: now reaches J7.2 (Pin_2)
- net BANK0_IOT.48b: now reaches J7.21 (Pin_21)
- net BANK0_IOT.49a: now reaches J7.23 (Pin_23)
- net BANK0_IOT.50b: now reaches J7.25 (Pin_25)
- net BANK0_IOT.51a: now reaches J7.27 (Pin_27)
- net BANK2_IOB.0a: now reaches J7.29 (Pin_29)
- net BANK0_IOT.37a: now reaches J7.3 (Pin_3)
- net FPGA.CDONE: now reaches J7.30 (Pin_30)
- net BANK2_IOB.2a: now reaches J7.31 (Pin_31)
- net FPGA.~{CRESET}: now reaches J7.32 (Pin_32)
- net BANK2_IOB.3b: now reaches J7.33 (Pin_33)
- net BANK2_IOB.4a: now reaches J7.35 (Pin_35)
- net BANK2_IOB.5b: now reaches J7.37 (Pin_37)
- net BANK2_IOB.6a: now reaches J7.39 (Pin_39)
- net BANK1_IOB.16a: now reaches J7.4 (Pin_4)
- net BANK2_IOB.8a: now reaches J7.41 (Pin_41)
- net BANK2_IOB.9b: now reaches J7.43 (Pin_43)
- net BANK0_IOT.38b: now reaches J7.5 (Pin_5)
- net BANK1_IOB.18a: now reaches J7.6 (Pin_6)
- net BANK0_IOT.39a: now reaches J7.7 (Pin_7)
- net BANK1_IOB.20a: now reaches J7.8 (Pin_8)
- net BANK0_IOT.41a: now reaches J7.9 (Pin_9)
- net PB6 renamed PB.6
- net PG15 renamed PG.15
- net PG2 renamed PG.2
- net PG3 renamed PG.3
- net PG4 renamed PG.4
- net PG5 renamed PG.5
- net PH5 renamed PH.5
- net PH6 renamed PH.6
- net PH7 renamed PH.7
- net PI12 renamed PI.12
- net PI13 renamed PI.13
- net PJ11 renamed PJ.11
- net PJ9 renamed PJ.9
- net PK2 renamed PK.2
- new net PF.2: J8.5 (Pin_5)
Other:
- note added: "FPGA GPIO"
- note added: "MCU GPIO"
- moved on the sheet: J7, J8
