File: kicad/mcu.kicad_sch (KiCad schematic)
At the start: 16 parts, among them U3 STM32H743XIHx, X1 25MHz, X2 32.768KHz

Commit message: many updates
Parts:
- C10, C11, C2, C3, C4, C5, C6, C7, C8, C9: footprint (none) -> Capacitor_SMD:C_0603_1608Metric
- R5, R6: footprint (none) -> Resistor_SMD:R_0603_1608Metric
- X1, X2: footprint (none) -> Crystal_AKL:Crystal_SMD_3225-4Pin_3.2x2.5mm
- renumbered TP2 to TP1
Connections:
- net HDMI_CEC: no longer names the net of U3.B5 (PB6)
Other:
- note added: "check crystal caps"
Changed lines of the file:
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@@
 		)
 	)
+	(text "check crystal caps"
+		(exclude_from_sim no)
+		(at 560.832 135.636 0)
+		(effects
+			(font
+				(size 1.27 1.27)
+			)
+		)
+	)
 	(text "RMII"
 		(exclude_from_sim no)
@@
 		)
 	)
+	(bus
+		(pts
+			(xy 386.08 137.16) (xy 384.81 137.16)
+		)
+		(stroke
+			(width 0)
+			(type default)
+		)
+	)
 	(wire
 		(pts
@@
 		)
 	)
+	(bus
+		(pts
+			(xy 386.08 149.86) (xy 384.81 149.86)
+		)
+		(stroke
+			(width 0)
+			(type default)
+		)
+	)
 	(wire
 		(pts
@@
 		)
 	)
-	(bus
-		(pts
-			(xy 386.08 154.94) (xy 386.08 134.62)
-		)
-		(stroke
-			(width 0)
-			(type default)
-		)
-	)
 	(wire
 		(pts
@@
 		)
 	)
-	(bus
-		(pts
-			(xy 384.81 134.62) (xy 386.08 134.62)
-		)
-		(stroke
-			(width 0)
-			(type default)
-		)
-	)
 	(wire
 		(pts
@@
 		)
 	)
+	(bus
+		(pts
+			(xy 386.08 147.32) (xy 386.08 137.16)
+		)
+		(stroke
+			(width 0)
+			(type default)
+		)
+	)
 	(wire
 		(pts
@@
 	(bus
 		(pts
+			(xy 386.08 154.94) (xy 386.08 149.86)
+		)
+		(stroke
+			(width 0)
+			(type default)
+		)
+	)
+	(bus
+		(pts
 			(xy 548.64 264.16) (xy 549.91 264.16)
 		)
@@
 	(wire
 		(pts
-			(xy 199.39 157.48) (xy 215.9 157.48)
-		)
-		(stroke
-			(width 0)
-			(type default)
-		)
-	)
-	(wire
-		(pts
 			(xy 482.6 187.96) (xy 495.3 187.96)
 		)
@@
 		)
 	)
-	(hierarchical_label "HDMI_CEC"
-		(shape input)
-		(at 215.9 157.48 0)
-		(effects
-			(font
-				(size 1.27 1.27)
-			)
-			(justify left)
-		)
-	)
 	(hierarchical_label "COMP2{INP INN}"
 		(shape bidirectional)
@@
 	)
 	(hierarchical_label "I2S2{MCK WS CK SDI SDO}"
-		(shape input)
+		(shape output)
 		(at 551.18 69.85 180)
 		(effects
@@
 		)
 	)
+	(hierarchical_label "RMII{TXD0 TXD1 TXEN RXD0 RXD1}"
+		(shape bidirectional)
+		(at 384.81 137.16 180)
+		(effects
+			(font
+				(size 1.27 1.27)
+			)
+			(justify right)
+		)
+	)
 	(hierarchical_label "SDMMC{D_{[0..4]} CLK CMD}"
 		(shape bidirectional)
@@
 	)
 	(hierarchical_label "SAI1A{MCLK FS SCK SD}"
-		(shape input)
+		(shape output)
 		(at 549.91 34.29 180)
 		(effects
@@
 	)
 	(hierarchical_label "SPI1{NSS SCK MISO MOSI}"
-		(shape input)
+		(shape bidirectional)
 		(at 382.27 224.79 180)
 		(effects
@@
 		)
 	)
-	(hierarchical_label "RMII{TXD0 TXD1 TXEN RXD0 RXD1 CRS_DV MDIO MDC}"
-		(shape bidirectional)
-		(at 384.81 134.62 180)
-		(effects
-			(font
-				(size 1.27 1.27)
-			)
-			(justify right)
-		)
-	)
 	(hierarchical_label "FDCAN1{RX TX}"
 		(shape bidirectional)
@@
 		)
 	)
+	(hierarchical_label "RMII{CRS_DV MDIO MDC}"
+		(shape bidirectional)
+		(at 384.81 149.86 180)
+		(effects
+			(font
+				(size 1.27 1.27)
+			)
+			(justify right)
+		)
+	)
 	(hierarchical_label "USB_OTG_FS{D- D+}"
 		(shape bidirectional)
@@
 	)
 	(hierarchical_label "DAC1_OUT1"
-		(shape input)
+		(shape output)
 		(at 215.9 109.22 0)
 		(effects
@@
 	)
 	(hierarchical_label "QUADSPI{D[4..0] CLK ~{CS}}"
-		(shape input)
+		(shape bidirectional)
 		(at 485.14 119.38 180)
 		(effects
@@
 			)
 		)
-		(property "Footprint" ""
+		(property "Footprint" "Capacitor_SMD:C_0603_1608Metric"
 			(at 558.8 118.11 0)
 			(hide yes)
@@
 			)
 		)
-		(property "Footprint" ""
+		(property "Footprint" "Capacitor_SMD:C_0603_1608Metric"
 			(at 92.71 322.58 0)
 			(hide yes)
@@
 			)
 		)
-		(property "Footprint" ""
+		(property "Footprint" "Resistor_SMD:R_0603_1608Metric"
 			(at 38.1 88.9 0)
 			(hide yes)
@@
 			)
 		)
-		(property "Footprint" ""
+		(property "Footprint" "Capacitor_SMD:C_0603_1608Metric"
 			(at 38.1 114.3 0)
 			(hide yes)
@@
 			)
 		)
-		(property "Footprint" ""
+		(property "Footprint" "Capacitor_SMD:C_0603_1608Metric"
 			(at 82.55 322.58 0)
 			(hide yes)
@@
 		(dnp no)
 		(fields_autoplaced yes)
-		(property "Reference" "TP2"
+		(property "Reference" "TP1"
 			(at 60.198 99.06 90)
 			(show_name no)
@@
 			(project "STM32H743"
 				(path "/f3410568-889b-492f-907e-34c84712a8ea/5a1d56ac-f234-404b-997d-39ebf9479f62"
-					(reference "TP2")
+					(reference "TP1")
 					(unit 1)
 				)
@@
 			)
 		)
-		(property "Footprint" ""
+		(property "Footprint" "Capacitor_SMD:C_0603_1608Metric"
 			(at 533.4 118.11 0)
 			(hide yes)
@@
 			)
 		)
-		(property "Footprint" ""
+		(property "Footprint" "Capacitor_SMD:C_0603_1608Metric"
 			(at 558.8 156.21 0)
 			(hide yes)
@@
 			)
 		)
-		(property "Footprint" ""
+		(property "Footprint" "Resistor_SMD:R_0603_1608Metric"
 			(at 50.8 88.9 0)
 			(hide yes)
@@
 			)
 		)
-		(property "Footprint" ""
+		(property "Footprint" "Crystal_AKL:Crystal_SMD_3225-4Pin_3.2x2.5mm"
 			(at 546.1 152.4 0)
 			(hide yes)
@@
 			)
 		)
-		(property "Footprint" ""
+		(property "Footprint" "Crystal_AKL:Crystal_SMD_3225-4Pin_3.2x2.5mm"
 			(at 546.1 114.3 0)
 			(hide yes)
@@
 			)
 		)
-		(property "Footprint" ""
+		(property "Footprint" "Capacitor_SMD:C_0603_1608Metric"
 			(at 50.8 114.3 0)
 			(hide yes)
@@
 			)
 		)
-		(property "Footprint" ""
+		(property "Footprint" "Capacitor_SMD:C_0603_1608Metric"
 			(at 71.12 322.58 0)
 			(hide yes)
@@
 			)
 		)
-		(property "Footprint" ""
+		(property "Footprint" "Capacitor_SMD:C_0603_1608Metric"
 			(at 533.4 156.21 0)
 			(hide yes)
@@
 			)
 		)
-		(property "Footprint" ""
+		(property "Footprint" "Capacitor_SMD:C_0603_1608Metric"
 			(at 63.5 114.3 0)
 			(hide yes)

Commit message: school wifi broken
Parts:
- added C64, C65, C66, C67, C68, C69, C70, C71, C72: 0.1uF, Capacitor_SMD:C_0603_1608Metric, symbol Device:C_Small
- added SW1, SW2: SW_Push, Button_Switch_SMD:Panasonic_EVQPUM_EVQPUD, symbol Switch:SW_Push
Connections:
- net +3.3V: now also C64.1, C65.1, C66.1, C67.1, C68.1, C69.1, C70.1, C71.1, C72.1
- net BOOT0: now also C2.1, R5.2, SW2.2; no longer C3.1, R6.2
- net GND: now also C64.2, C65.2, C66.2, C67.2, C68.2, C69.2, C70.2, C71.2, C72.2, SW1.1, SW2.1
- net NRST: now also C3.1, R6.2, SW1.2; no longer C2.1, R5.2
- net ~{SD_DET}: now reaches U3.A12 (PD4)
- net PB6: now reaches U3.B5 (PB6)
- net ~{RMII_RST}: now reaches U3.D3 (PE3)
- net PG15: now reaches U3.D6 (PG15)
- net PF2: now reaches U3.G1 (PF2)
- net PG5: now reaches U3.G14 (PG5)
- net PI12: now reaches U3.H1 (PI12)
- net PG4: now reaches U3.H14 (PG4)
- net PG3: now reaches U3.H15 (PG3)
- net PG2: now reaches U3.H16 (PG2)
- net PK2: now reaches U3.H17 (PK2)
- net PI13: now reaches U3.H2 (PI13)
- net PJ11: now reaches U3.K14 (PJ11)
- net PJ9: now reaches U3.M14 (PJ9)
- net FPGA.~{CRESET}: now reaches U3.P15 (PD15)
- net FPGA.CDONE: now reaches U3.P16 (PD14)
- net PH5: now reaches U3.P4 (PH5)
- net FPGA_ACT: now reaches U3.P8 (PF14)
- net MCU_ACT: now reaches U3.R11 (PE15)
- net ULPI_RESET: now reaches U3.R14 (PH12)
- net FPGA_FAULT: now reaches U3.R7 (PF12)
- net MCU_FAULT: now reaches U3.R9 (PF15)
- net PH6: now reaches U3.T11 (PH6)
- net 2.5V_EN: now reaches U3.T8 (PG0)
- net PH7: now reaches U3.U13 (PH7)
- net 1.2V_EN: now reaches U3.U7 (PJ4)
- net 1.8V_EN: now reaches U3.U8 (PG1)
- no-connect marks 0 -> 1
Other:
- note added: "FPGA configuration pins"
- note added: "RGB888"
- note removed: "confirm these"
- moved on the sheet: C2, C3, R5, R6

Commit message: blenders
Connections:
- net ~{SPI1.CS} is gone; now on net SPI1.NSS: U3.A14 (PA15)
- net PB6 renamed PB.6
- net PF2 renamed PF.2
- net PG15 renamed PG.15
- net PG2 renamed PG.2
- net PG3 renamed PG.3
- net PG4 renamed PG.4
- net PG5 renamed PG.5
- net PH5 renamed PH.5
- net PH6 renamed PH.6
- net PH7 renamed PH.7
- net PI12 renamed PI.12
- net PI13 renamed PI.13
- net PJ11 renamed PJ.11
- net PJ9 renamed PJ.9
- net PK2 renamed PK.2
Other:
- note added: "Spare GPIO"
- note added: "maybe these should be connected to the fpga directly but the mcu manages the fpga so it should be ok"
