File: kicad/STM32H743.kicad_pcb (KiCad board)
At the start: 6 copper layers, 50 x 75 mm, 126 parts, among them J1 USB_A, J2 USB_C_Receptacle_USB2.0_16P, J3 RJ45_Halo_HFJ11-x2450E-LxxRL, J4 Micro_SD_Card_Det2, J5 AudioJack3, J6 Conn_02x05_Counter_Clockwise, U1 USBLC6-2SC6, U10 TPD3S014, U11 USB3300-EZK, U12 ICE40UP5K-SG48ITR, U2 USBLC6-2SC6, U3 STM32H743XIHx, U4 TLV75733PDBV, U5 TLV75725PDBV, U6 TLV75718PDBV, U7 TLV75712PDBV, U8 LAN8742A, U9 CS4344, X1 25MHz, X2 32.768KHz, X3 TCXO, Y1 Si5351C-B-GM

Commit message: school wifi broken
Parts:
- added C100: 0.1uF, Capacitor_SMD:C_0603_1608Metric, F.Cu at (115.0, 66.0)
- added C101: 0.1uF, Capacitor_SMD:C_0603_1608Metric, F.Cu at (106.0, 77.5)
- added C64: 0.1uF, Capacitor_SMD:C_0603_1608Metric, F.Cu at (48.0, 57.0)
- added C65: 0.1uF, Capacitor_SMD:C_0603_1608Metric, F.Cu at (52.0, 57.0)
- added C66: 0.1uF, Capacitor_SMD:C_0603_1608Metric, F.Cu at (66.0, 61.0)
- added C67: 0.1uF, Capacitor_SMD:C_0603_1608Metric, F.Cu at (66.0, 65.0)
- added C68: 0.1uF, Capacitor_SMD:C_0603_1608Metric, F.Cu at (66.0, 71.0)
- added C69: 0.1uF, Capacitor_SMD:C_0603_1608Metric, F.Cu at (58.0, 80.0)
- added C70: 0.1uF, Capacitor_SMD:C_0603_1608Metric, F.Cu at (45.0, 69.0)
- added C71: 0.1uF, Capacitor_SMD:C_0603_1608Metric, B.Cu at (53.0, 67.5)
- added C72: 0.1uF, Capacitor_SMD:C_0603_1608Metric, B.Cu at (57.0, 67.5)
- added C73: 0.1uF, Capacitor_SMD:C_0603_1608Metric, F.Cu at (66.0, 97.0)
- added C92: 0.1uF, Capacitor_SMD:C_0603_1608Metric, F.Cu at (48.5, 48.0)
- added C93: 0.1uF, Capacitor_SMD:C_0603_1608Metric, F.Cu at (48.5, 49.5)
- added C94: 0.1uF, Capacitor_SMD:C_0603_1608Metric, F.Cu at (46.0, 55.5)
- added C95: 0.1uF, Capacitor_SMD:C_0603_1608Metric, F.Cu at (44.0, 55.5)
- added C96: 0.1uF, Capacitor_SMD:C_0603_1608Metric, F.Cu at (42.0, 55.5)
- added C97: 0.1uF, Capacitor_SMD:C_0603_1608Metric, F.Cu at (95.0, 65.0)
- added C98: 0.1uF, Capacitor_SMD:C_0603_1608Metric, F.Cu at (115.0, 64.0)
- added C99: 0.1uF, Capacitor_SMD:C_0603_1608Metric, F.Cu at (95.0, 63.0)
- added D10: RED, LED_SMD:LED_0603_1608Metric, F.Cu at (33.0, 97.0)
- added D11: LED_ABGR, LED_SMD:LED_Cree-PLCC4_2x2mm_CW, F.Cu at (115.0, 57.5)
- added D3: GREEN, LED_SMD:LED_0603_1608Metric, F.Cu at (94.0, 103.0)
- added D4: GREEN, LED_SMD:LED_0603_1608Metric, F.Cu at (96.0, 103.0)
- added D5: GREEN, LED_SMD:LED_0603_1608Metric, F.Cu at (98.0, 103.0)
- added D6: GREEN, LED_SMD:LED_0603_1608Metric, F.Cu at (100.0, 103.0)
- added D7: YELLOW, LED_SMD:LED_0603_1608Metric, F.Cu at (33.0, 91.0)
- added D8: RED, LED_SMD:LED_0603_1608Metric, F.Cu at (33.0, 93.0)
- added D9: YELLOW, LED_SMD:LED_0603_1608Metric, F.Cu at (33.0, 95.0)
- added G***: LOGO, customimages:linuxpenguin-mask, F.Cu at (61.0, 53.2)
- added G***: LOGO, customimages:linuxpenguin_cu, F.Cu at (61.0, 53.2)
- added H1: MountingHole, MountingHole:MountingHole_3.2mm_M3, F.Cu at (125.0, 35.0)
- added H2: MountingHole, MountingHole:MountingHole_3.2mm_M3, F.Cu at (125.0, 100.0)
- added J7: Conn_02x22_Odd_Even, Connector_PinSocket_2.54mm:PinSocket_2x22_P2.54mm_Vertical, F.Cu at (126.3, 40.8)
- added J8: Conn_02x10_Odd_Even, Connector_PinSocket_2.54mm:PinSocket_2x10_P2.54mm_Vertical, F.Cu at (93.6, 33.7)
- added MIC1: MMICT390200012, easyeda2kicad:MIC-SMD_5P-L3.5-W2.7-TL_MMICT390200012, F.Cu at (63.0, 97.0)
- added RN1: 1k, Resistor_SMD_AKL:R_Array_Concave_4x0603, F.Cu at (103.0, 101.0)
- added RN2: 1k, Resistor_SMD_AKL:R_Array_Concave_4x0603, F.Cu at (35.0, 100.0)
- added RN3: 0, Resistor_SMD_AKL:R_Array_Concave_4x0603, F.Cu at (103.0, 77.5)
- added SW1: SW_Push, Button_Switch_SMD:Panasonic_EVQPUM_EVQPUD, F.Cu at (32.0, 63.0)
- added SW2: SW_Push, Button_Switch_SMD:Panasonic_EVQPUM_EVQPUD, F.Cu at (32.0, 72.0)
- added TP3: TestPoint, TestPoint:TestPoint_Pad_D1.5mm, F.Cu at (80.0, 69.5)
- added TP4: TestPoint, TestPoint:TestPoint_Pad_D1.5mm, F.Cu at (78.0, 45.5)
- added TP5: TestPoint, TestPoint:TestPoint_Pad_D1.5mm, F.Cu at (82.0, 45.5)
- added TP6: TestPoint, TestPoint:TestPoint_Pad_D1.5mm, F.Cu at (85.0, 45.5)
- added TP7: TestPoint, TestPoint:TestPoint_Pad_D1.5mm, F.Cu at (92.0, 53.5)
- J4: footprint Connector_Card:microSD_HC_Molex_104031-0811 -> Connector_Card:microSD_HC_Hirose_DM3D-SF
- moved R6 149.4 mm to (32.0, 56.0)
- moved X1 142.8 mm to (39.7, 67.5), turned to 90 degrees
- moved R5 140.9 mm to (36.0, 78.0), turned to 180 degrees
- moved X2 140.5 mm to (44.0, 62.0), turned to 90 degrees
- moved C3 139.9 mm to (32.0, 58.0), turned to 180 degrees
- moved C10 138.4 mm to (39.7, 64.3)
- moved C2 136.5 mm to (32.0, 77.0), turned to 180 degrees
- moved C11 135.8 mm to (44.0, 58.8)
- moved C8 134.2 mm to (39.7, 70.7), turned to 180 degrees
- moved C9 131.6 mm to (44.0, 65.2), turned to 180 degrees
- moved C4 124.2 mm to (45.0, 76.0), turned to -90 degrees
- moved J1 122.2 mm to (76.5, 91.5)
- moved C5 120.4 mm to (54.0, 57.0), turned to 90 degrees
- moved C37 118.5 mm to (60.0, 32.0), turned to 90 degrees
- moved C7 116.6 mm to (56.0, 80.0), turned to -90 degrees
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Connections:
- net Net-(J3-RD+) renamed /Ethernet/RD+
- net Net-(J3-RD-) renamed /Ethernet/RD-
- net Net-(J3-TD+) renamed /Ethernet/TD+
- net Net-(J3-TD-) renamed /Ethernet/TD-
- C2 pad 1: /Connector/NRST -> /Connector/BOOT0
- C3 pad 1: /Connector/BOOT0 -> /Connector/NRST
- J4 pad 10: /uSD/~{SD_DET} -> /MCU/~{SD_DET}
- J5 pad R: unconnected-(J5-PadR) -> AOUTR
- J5 pad S: unconnected-(J5-PadS) -> GND
- J5 pad T: unconnected-(J5-PadT) -> AOUTL
- R12 pad 2: /uSD/~{SD_DET} -> /MCU/~{SD_DET}
- R27 pad 2: unconnected-(R27-Pad2) -> Net-(R27-Pad2)
- R28 pad 2: unconnected-(R28-Pad2) -> Net-(R28-Pad2)
- R30 pad 2: unconnected-(R30-Pad2) -> Net-(R30-Pad2)
- R31 pad 2: unconnected-(R31-Pad2) -> Net-(R31-Pad2)
- R32 pad 2: unconnected-(R32-Pad2) -> Net-(R32-Pad2)
- R5 pad 2: /Connector/NRST -> /Connector/BOOT0
- R6 pad 2: /Connector/BOOT0 -> /Connector/NRST
- U12 pad 14: /FPGA/SPI1.MISO -> Net-(RN3-R1.2)
- U12 pad 15: /FPGA/SPI1.SCK -> Net-(RN3-R2.2)
- U12 pad 16: /FPGA/SPI1.NSS -> Net-(RN3-R3.2)
- U12 pad 17: /FPGA/SPI1.MOSI -> Net-(RN3-R4.2)
- U12 pad 39: unconnected-(U12A-RGB0-Pad39) -> Net-(D11-RK)
- U12 pad 40: unconnected-(U12A-RGB1-Pad40) -> Net-(D11-GK)
- U12 pad 41: unconnected-(U12A-RGB2-Pad41) -> Net-(D11-BK)
- U3 pad A12: unconnected-(U3-PD4-PadA12) -> /MCU/~{SD_DET}
- U3 pad B5: unconnected-(U3-PB6-PadB5) -> /GPIO/PB6
- U3 pad D3: unconnected-(U3-PE3-PadD3) -> /Ethernet/~{RMII_RST}
- U3 pad D6: unconnected-(U3-PG15-PadD6) -> /GPIO/PG15
- U3 pad G1: unconnected-(U3-PF2-PadG1) -> /GPIO/PF2
- U3 pad G14: unconnected-(U3-PG5-PadG14) -> /GPIO/PG5
- U3 pad H1: unconnected-(U3-PI12-PadH1) -> /GPIO/PI12
- U3 pad H14: unconnected-(U3-PG4-PadH14) -> /GPIO/PG4
- U3 pad H15: unconnected-(U3-PG3-PadH15) -> /GPIO/PG3
- U3 pad H16: unconnected-(U3-PG2-PadH16) -> /GPIO/PG2
- U3 pad H17: unconnected-(U3-PK2-PadH17) -> /GPIO/PK2
- U3 pad H2: unconnected-(U3-PI13-PadH2) -> /GPIO/PI13
- U3 pad K14: unconnected-(U3-PJ11-PadK14) -> /GPIO/PJ11
- U3 pad M14: unconnected-(U3-PJ9-PadM14) -> /GPIO/PJ9
- U3 pad P15: unconnected-(U3-PD15-PadP15) -> /FPGA/FPGA.~{CRESET}
- U3 pad P16: unconnected-(U3-PD14-PadP16) -> /FPGA/FPGA.CDONE
- U3 pad P4: unconnected-(U3-PH5-PadP4) -> /GPIO/PH5
- U3 pad P8: unconnected-(U3-PF14-PadP8) -> /LEDs/FPGA_ACT
- U3 pad R1: /MCU/DFSDM1.CKIN1 -> /Audio/DFSDM1.CKIN1
- U3 pad R11: unconnected-(U3-PE15-PadR11) -> /LEDs/MCU_ACT
- U3 pad R14: unconnected-(U3-PH12-PadR14) -> ~{ULPI_RESET}
- U3 pad R2: /MCU/DFSDM1.DATIN1 -> /Audio/DFSDM1.DATIN1
- U3 pad R7: unconnected-(U3-PF12-PadR7) -> /LEDs/FPGA_FAULT
- U3 pad R9: unconnected-(U3-PF15-PadR9) -> /LEDs/MCU_FAULT
- U3 pad T11: unconnected-(U3-PH6-PadT11) -> /GPIO/PH6
- U3 pad T8: unconnected-(U3-PG0-PadT8) -> /MCU/2.5V_EN
- U3 pad U13: unconnected-(U3-PH7-PadU13) -> /GPIO/PH7
- U3 pad U7: unconnected-(U3-PJ4-PadU7) -> /MCU/1.2V_EN
- U3 pad U8: unconnected-(U3-PG1-PadU8) -> /MCU/1.8V_EN
- U5 pad 3: /Power/2.5V_EN -> /MCU/2.5V_EN
- U6 pad 3: /Power/1.8V_EN -> /MCU/1.8V_EN
- U7 pad 3: /Power/1.2V_EN -> /MCU/1.2V_EN
Routing:
- net +5V: track 26.5 -> 168.3 mm, vias 4 -> 7
- net +3.3V: track 2.34 -> 142.5 mm, vias 12 -> 46
- net GND: track 26.6 -> 161.4 mm, vias 22 -> 151
- net +1.2V: track 0.00 -> 85.3 mm, vias 0 -> 4
- net /Clock/ETH_CLK: track 0.00 -> 70.2 mm, vias 0 -> 2
- net +2.5V: track 0.00 -> 69.2 mm, vias 0 -> 3
- net /FPGA/SPI1.SCK: track 0.57 -> 65.7 mm, vias 1 -> 2
- net /FPGA/SPI1.MISO: track 0.00 -> 63.1 mm, vias 0 -> 2
- net /FPGA/SPI1.MOSI: track 0.57 -> 62.0 mm, vias 1 -> 2
- net /MCU/1.2V_EN: track 0.00 -> 57.7 mm, vias 0 -> 5
- net +3.3VFPGA: track 0.00 -> 56.4 mm, vias 0 -> 4
- net /MCU/HS_ULPI.DIR: track 0.57 -> 55.8 mm, vias 1 -> 3
- net /Connector/BOOT0: track 0.00 -> 53.8 mm, vias 0 -> 5
- net /MCU/1.8V_EN: track 0.00 -> 53.5 mm, vias 0 -> 5
- net /Audio/SAI2B.SD: track 0.00 -> 53.1 mm, vias 0 -> 3
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- added copper zone on B.Cu, net +3.3V
- added copper zone on In2.Cu, net +3.3V
- added copper zone on B.Cu, net GND
- added copper zone on In2.Cu, net GND
- added copper zone on In3.Cu, net GND
- added copper zone on In4.Cu, net GND
Other:
- board size 50 x 75 mm -> 100 x 75 mm
- board text added: "1.2V"
- board text added: "1.8V"
- board text added: "2.5V"
- board text added: "3.3V"
- board text added: "5V"
- board text added: "ACT"
- board text added: "CLK3"
- board text added: "CLK4"
- board text added: "CLK5"
- board text added: "CLK6"
- board text added: "CLK7"
- board text added: "FAULT"
- board text added: "FPGA"
- board text added: "GND"
- board text added: "MCU"
- board text added: "STM32H743XIH6"
- board text added: "VREF+"
- board text added: "iCE40UP5K"
- board text added: "~{ULPI_RESET}"

Commit message: blenders
Parts:
- added J9: Conn_02x05_Odd_Even, Connector_PinHeader_2.54mm:PinHeader_2x05_P2.54mm_Vertical, F.Cu at (49.9, 84.5)
- moved G*** 4.46 mm to (65.5, 53.2) (x2)
- moved C69 1.50 mm to (58.0, 78.5)
- moved C7 1.50 mm to (56.0, 78.5)
Connections:
- net /GPIO/PB6 renamed /GPIO/PB.6
- net /GPIO/PF2 renamed /GPIO/PF.2
- net /GPIO/PG15 renamed /GPIO/PG.15
- net /GPIO/PG2 renamed /GPIO/PG.2
- net /GPIO/PG3 renamed /GPIO/PG.3
- net /GPIO/PG4 renamed /GPIO/PG.4
- net /GPIO/PG5 renamed /GPIO/PG.5
- net /GPIO/PH5 renamed /GPIO/PH.5
- net /GPIO/PH6 renamed /GPIO/PH.6
- net /GPIO/PH7 renamed /GPIO/PH.7
- net /GPIO/PI12 renamed /GPIO/PI.12
- net /GPIO/PI13 renamed /GPIO/PI.13
- net /GPIO/PJ11 renamed /GPIO/PJ.11
- net /GPIO/PJ9 renamed /GPIO/PJ.9
- net /GPIO/PK2 renamed /GPIO/PK.2
- J7 pad 1: unconnected-(J7-Pin_1-Pad1) -> /FPGA/BANK0_IOT.36b
- J7 pad 10: unconnected-(J7-Pin_10-Pad10) -> /FPGA/BANK1_IOB.22a
- J7 pad 11: unconnected-(J7-Pin_11-Pad11) -> /FPGA/BANK0_IOT.42b
- J7 pad 12: unconnected-(J7-Pin_12-Pad12) -> /FPGA/BANK1_IOB.23b
- J7 pad 13: unconnected-(J7-Pin_13-Pad13) -> /FPGA/BANK0_IOT.43a
- J7 pad 14: unconnected-(J7-Pin_14-Pad14) -> /FPGA/BANK1_IOB.24a
- J7 pad 15: unconnected-(J7-Pin_15-Pad15) -> /FPGA/BANK0_IOT.44b
- J7 pad 16: unconnected-(J7-Pin_16-Pad16) -> /FPGA/BANK1_IOB.29b
- J7 pad 17: unconnected-(J7-Pin_17-Pad17) -> /FPGA/BANK0_IOT.45a
- J7 pad 18: unconnected-(J7-Pin_18-Pad18) -> /FPGA/BANK1_IOB.31b
- J7 pad 19: unconnected-(J7-Pin_19-Pad19) -> /FPGA/BANK0_IOT.46b
- J7 pad 2: unconnected-(J7-Pin_2-Pad2) -> /FPGA/BANK1_IOB.13b
- J7 pad 20: unconnected-(J7-Pin_20-Pad20) -> +3.3V
- J7 pad 21: unconnected-(J7-Pin_21-Pad21) -> /FPGA/BANK0_IOT.48b
- J7 pad 22: unconnected-(J7-Pin_22-Pad22) -> +3.3V
- J7 pad 23: unconnected-(J7-Pin_23-Pad23) -> /FPGA/BANK0_IOT.49a
- J7 pad 24: unconnected-(J7-Pin_24-Pad24) -> +3.3V
- J7 pad 25: unconnected-(J7-Pin_25-Pad25) -> /FPGA/BANK0_IOT.50b
- J7 pad 26: unconnected-(J7-Pin_26-Pad26) -> +3.3V
- J7 pad 27: unconnected-(J7-Pin_27-Pad27) -> /FPGA/BANK0_IOT.51a
- J7 pad 28: unconnected-(J7-Pin_28-Pad28) -> +3.3V
- J7 pad 29: unconnected-(J7-Pin_29-Pad29) -> /FPGA/BANK2_IOB.0a
- J7 pad 3: unconnected-(J7-Pin_3-Pad3) -> /FPGA/BANK0_IOT.37a
- J7 pad 30: unconnected-(J7-Pin_30-Pad30) -> /FPGA/FPGA.CDONE
- J7 pad 31: unconnected-(J7-Pin_31-Pad31) -> /FPGA/BANK2_IOB.2a
- J7 pad 32: unconnected-(J7-Pin_32-Pad32) -> /FPGA/FPGA.~{CRESET}
- J7 pad 33: unconnected-(J7-Pin_33-Pad33) -> /FPGA/BANK2_IOB.3b
- J7 pad 34: unconnected-(J7-Pin_34-Pad34) -> GND
- J7 pad 35: unconnected-(J7-Pin_35-Pad35) -> /FPGA/BANK2_IOB.4a
- J7 pad 36: unconnected-(J7-Pin_36-Pad36) -> GND
- J7 pad 37: unconnected-(J7-Pin_37-Pad37) -> /FPGA/BANK2_IOB.5b
- J7 pad 38: unconnected-(J7-Pin_38-Pad38) -> GND
- J7 pad 39: unconnected-(J7-Pin_39-Pad39) -> /FPGA/BANK2_IOB.6a
- J7 pad 4: unconnected-(J7-Pin_4-Pad4) -> /FPGA/BANK1_IOB.16a
- J7 pad 40: unconnected-(J7-Pin_40-Pad40) -> GND
- J7 pad 41: unconnected-(J7-Pin_41-Pad41) -> /FPGA/BANK2_IOB.8a
- J7 pad 42: unconnected-(J7-Pin_42-Pad42) -> GND
- J7 pad 43: unconnected-(J7-Pin_43-Pad43) -> /FPGA/BANK2_IOB.9b
- J7 pad 44: unconnected-(J7-Pin_44-Pad44) -> GND
- J7 pad 5: unconnected-(J7-Pin_5-Pad5) -> /FPGA/BANK0_IOT.38b
- J7 pad 6: unconnected-(J7-Pin_6-Pad6) -> /FPGA/BANK1_IOB.18a
- J7 pad 7: unconnected-(J7-Pin_7-Pad7) -> /FPGA/BANK0_IOT.39a
- J7 pad 8: unconnected-(J7-Pin_8-Pad8) -> /FPGA/BANK1_IOB.20a
- J7 pad 9: unconnected-(J7-Pin_9-Pad9) -> /FPGA/BANK0_IOT.41a
- U12 pad 10: unconnected-(U12B-IOB_18a-Pad10) -> /FPGA/BANK1_IOB.18a
- U12 pad 11: unconnected-(U12B-IOB_20a-Pad11) -> /FPGA/BANK1_IOB.20a
- U12 pad 12: unconnected-(U12B-IOB_22a-Pad12) -> /FPGA/BANK1_IOB.22a
- U12 pad 13: unconnected-(U12B-IOB_24a-Pad13) -> /FPGA/BANK1_IOB.24a
- U12 pad 18: unconnected-(U12B-IOB_31b-Pad18) -> /FPGA/BANK1_IOB.31b
- U12 pad 19: unconnected-(U12B-IOB_29b-Pad19) -> /FPGA/BANK1_IOB.29b
- U12 pad 2: unconnected-(U12C-IOB_6a-Pad2) -> /FPGA/BANK2_IOB.6a
- U12 pad 21: unconnected-(U12B-IOB_23b-Pad21) -> /FPGA/BANK1_IOB.23b
- U12 pad 23: unconnected-(U12A-IOT_37a-Pad23) -> /FPGA/BANK0_IOT.37a
- U12 pad 25: unconnected-(U12A-IOT_36b-Pad25) -> /FPGA/BANK0_IOT.36b
- U12 pad 26: unconnected-(U12A-IOT_39a-Pad26) -> /FPGA/BANK0_IOT.39a
- U12 pad 27: unconnected-(U12A-IOT_38b-Pad27) -> /FPGA/BANK0_IOT.38b
- U12 pad 28: unconnected-(U12A-IOT_41a-Pad28) -> /FPGA/BANK0_IOT.41a
- U12 pad 3: unconnected-(U12C-IOB_9b-Pad3) -> /FPGA/BANK2_IOB.9b
- U12 pad 31: unconnected-(U12A-IOT_42b-Pad31) -> /FPGA/BANK0_IOT.42b
- U12 pad 32: unconnected-(U12A-IOT_43a-Pad32) -> /FPGA/BANK0_IOT.43a
- U12 pad 34: unconnected-(U12A-IOT_44b-Pad34) -> /FPGA/BANK0_IOT.44b
- U12 pad 35: unconnected-(U12A-IOT_46b_G0-Pad35) -> /FPGA/BANK0_IOT.46b
- U12 pad 36: unconnected-(U12A-IOT_48b-Pad36) -> /FPGA/BANK0_IOT.48b
- U12 pad 37: unconnected-(U12A-IOT_45a_G1-Pad37) -> /FPGA/BANK0_IOT.45a
- U12 pad 38: unconnected-(U12A-IOT_50b-Pad38) -> /FPGA/BANK0_IOT.50b
- U12 pad 4: unconnected-(U12C-IOB_8a-Pad4) -> /FPGA/BANK2_IOB.8a
- U12 pad 42: unconnected-(U12A-IOT_51a-Pad42) -> /FPGA/BANK0_IOT.51a
- U12 pad 43: unconnected-(U12A-IOT_49a-Pad43) -> /FPGA/BANK0_IOT.49a
- U12 pad 44: unconnected-(U12C-IOB_3b_G6-Pad44) -> /FPGA/BANK2_IOB.3b
- U12 pad 45: unconnected-(U12C-IOB_5b-Pad45) -> /FPGA/BANK2_IOB.5b
- U12 pad 46: unconnected-(U12C-IOB_0a-Pad46) -> /FPGA/BANK2_IOB.0a
- U12 pad 47: unconnected-(U12C-IOB_2a-Pad47) -> /FPGA/BANK2_IOB.2a
- U12 pad 48: unconnected-(U12C-IOB_4a-Pad48) -> /FPGA/BANK2_IOB.4a
- U12 pad 6: unconnected-(U12B-IOB_13b-Pad6) -> /FPGA/BANK1_IOB.13b
- U12 pad 9: unconnected-(U12B-IOB_16a-Pad9) -> /FPGA/BANK1_IOB.16a
- U3 pad A14: /MCU/~{SPI1.CS} -> /FPGA/SPI1.NSS
- U3 pad B14: /Connector/SWD.SWCLK -> SWCLK
- U3 pad C15: /Connector/SWD.SWDIO -> SWDIO
Routing:
- net /GPIO/PH.6: track 7.28 -> 74.5 mm, vias 1 -> 3
- net /GPIO/PH.7: track 10.2 -> 77.2 mm, vias 1 -> 4
- net /GPIO/PG.2: track 12.7 -> 74.4 mm, vias 1 -> 3
- net /GPIO/PF.2: track 10.3 -> 71.2 mm, vias 2 -> 3
- net /GPIO/PI.12: track 13.8 -> 74.5 mm, vias 2 -> 4
- net /FPGA/SPI1.NSS: track 0.92 -> 60.7 mm, vias 1 -> 3
- net /GPIO/PI.13: track 16.7 -> 76.4 mm, vias 2 -> 4
- net /GPIO/PJ.9: track 19.7 -> 78.2 mm, vias 2 -> 3
- net /GPIO/PG.3: track 16.3 -> 73.8 mm, vias 2 -> 3
- net /GPIO/PG.4: track 19.2 -> 74.7 mm, vias 2 -> 4
- net /GPIO/PG.5: track 22.1 -> 76.0 mm, vias 2 -> 3
- net /GPIO/PG.15: track 25.0 -> 78.9 mm, vias 2 -> 4
- net /GPIO/PJ.11: track 22.6 -> 76.3 mm, vias 2 -> 4
- net /GPIO/PK.2: track 25.3 -> 76.8 mm, vias 1 -> 3
- net /FPGA/BANK2_IOB.9b: track 0.00 -> 49.2 mm, vias 0 -> 1
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
Commit message: blender
Other:
- board text added: "B_0a"
- board text added: "B_13b"
- board text added: "B_16a"
- board text added: "B_18a"
- board text added: "B_20a"
- board text added: "B_22a"
- board text added: "B_23b"
- board text added: "B_24a"
- board text added: "B_29b"
- board text added: "B_2a"
- board text added: "B_31b"
- board text added: "B_3b"
- board text added: "B_4a"
- board text added: "B_5b"
- board text added: "B_6a"
- board text added: "B_8a"
- board text added: "B_9b"
- board text added: "DONE"
- board text added: "PB6"
- board text added: "PF2"
- board text added: "PG15"
- board text added: "PG2"
- board text added: "PG3"
- board text added: "PG4"
- board text added: "PG5"
- board text added: "RESET"
- board text added: "T_36b"
- board text added: "T_37a"
- board text added: "T_38b"
- board text added: "T_39a"
- board text added: "T_41a"
- board text added: "T_42b"
- board text added: "T_43a"
- board text added: "T_44b"
- board text added: "T_45a"
- board text added: "T_46b"
- board text added: "T_48b"
- board text added: "T_49a"
- board text added: "T_50b"
- board text added: "T_51a"

Commit message: rendering
Other:
- board text added: "PH5"
- board text added: "PH6"
- board text added: "PH7"
- board text added: "PI12"
- board text added: "PI13"
- board text added: "PJ11"
- board text added: "PJ9"
- board text added: "PK2"
Changed lines of the file:
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@@
 		(tags "LED Cree PLCC-4 2020 CLMVB-FKA CLMVC-FKA")
 		(property "Reference" "D11"
-			(at 0 -2.25 0)
+			(at 0 -1.6 0)
 			(layer "F.SilkS")
 			(effects
 				(font
-					(size 1 1)
-					(thickness 0.15)
+					(size 0.5 0.5)
+					(thickness 0.1)
+					(bold yes)
 				)
 			)
@@
 		(tags "Through hole pin header THT 2x05 2.54mm double row")
 		(property "Reference" "J9"
-			(at 1.27 -2.380001 90)
+			(at 1.27 -2.02 90)
 			(layer "F.SilkS")
 			(effects
 				(font
-					(size 1 1)
-					(thickness 0.15)
+					(size 0.5 0.5)
+					(thickness 0.1)
+					(bold yes)
 				)
 			)
@@
 		)
 	)
+	(gr_text "3.3V"
+		(at 93.6 38 90)
+		(layer "F.SilkS")
+		(effects
+			(font
+				(size 0.5 0.5)
+				(thickness 0.1)
+				(bold yes)
+			)
+			(justify right)
+		)
+	)
+	(gr_text "PH5"
+		(at 96.1 38 90)
+		(layer "F.SilkS")
+		(effects
+			(font
+				(size 0.5 0.5)
+				(thickness 0.1)
+				(bold yes)
+			)
+			(justify right)
+		)
+	)
+	(gr_text "PH6"
+		(at 98.7 38 90)
+		(layer "F.SilkS")
+		(effects
+			(font
+				(size 0.5 0.5)
+				(thickness 0.1)
+				(bold yes)
+			)
+			(justify right)
+		)
+	)
+	(gr_text "PH7"
+		(at 101.2 38 90)
+		(layer "F.SilkS")
+		(effects
+			(font
+				(size 0.5 0.5)
+				(thickness 0.1)
+				(bold yes)
+			)
+			(justify right)
+		)
+	)
+	(gr_text "PI12"
+		(at 103.7 38 90)
+		(layer "F.SilkS")
+		(effects
+			(font
+				(size 0.5 0.5)
+				(thickness 0.1)
+				(bold yes)
+			)
+			(justify right)
+		)
+	)
+	(gr_text "PI13"
+		(at 106.3 38 90)
+		(layer "F.SilkS")
+		(effects
+			(font
+				(size 0.5 0.5)
+				(thickness 0.1)
+				(bold yes)
+			)
+			(justify right)
+		)
+	)
+	(gr_text "PJ9"
+		(at 108.8 38 90)
+		(layer "F.SilkS")
+		(effects
+			(font
+				(size 0.5 0.5)
+				(thickness 0.1)
+				(bold yes)
+			)
+			(justify right)
+		)
+	)
+	(gr_text "PJ11"
+		(at 111.3 38 90)
+		(layer "F.SilkS")
+		(effects
+			(font
+				(size 0.5 0.5)
+				(thickness 0.1)
+				(bold yes)
+			)
+			(justify right)
+		)
+	)
+	(gr_text "PK2"
+		(at 113.9 38 90)
+		(layer "F.SilkS")
+		(effects
+			(font
+				(size 0.5 0.5)
+				(thickness 0.1)
+				(bold yes)
+			)
+			(justify right)
+		)
+	)
+	(gr_text "GND"
+		(at 116.5 38 90)
+		(layer "F.SilkS")
+		(effects
+			(font
+				(size 0.5 0.5)
+				(thickness 0.1)
+				(bold yes)
+			)
+			(justify right)
+		)
+	)
